File: DrillPowerSupply.kicad_pcb (KiCad board)
At the start: 4 copper layers, 69 x 55 mm, 11 parts, among them J1 1711026, J2 1711039, J3 90136-2104, U1 NE555P

Commit message: PCB done
Parts:
- added H1: MountingHole, MountingHole:MountingHole_3.2mm_M3_Pad_Via, F.Cu at (113.5, 61.9)
- added H2: MountingHole, MountingHole:MountingHole_3.2mm_M3_Pad_Via, F.Cu at (166.7, 62.2)
- added H3: MountingHole, MountingHole:MountingHole_3.2mm_M3_Pad_Via, F.Cu at (113.2, 106.8)
- added H4: MountingHole, MountingHole:MountingHole_3.2mm_M3_Pad_Via, F.Cu at (166.5, 106.6)
- moved J1 3.19 mm to (114.0, 72.2)
- moved J2 1.00 mm to (114.0, 89.0)
Routing:
- net Net-(D2-A): track 18.7 -> 72.2 mm
- net +5V: track 25.3 -> 77.1 mm
- net Net-(U1-Q): track 15.0 -> 30.3 mm
- net Net-(U1-THR): track 39.7 -> 46.9 mm
- net Net-(D1-A): track 26.2 -> 28.7 mm
- net Net-(D1-K): track 17.0 -> 15.9 mm
Other:
- board text added: "Drill Spindle PWM Controller Bernd Prager V0.0.5 04/07/2025"
