File: DrillPowerSupply.kicad_sch (KiCad schematic)
At the start: 11 parts, among them J1 1711026, J2 1711039, J3 90136-2104, U1 NE555P

Commit message: PCB done
Parts:
- added H1, H2, H3, H4: MountingHole, MountingHole:MountingHole_3.2mm_M3_Pad_Via, symbol Mechanical:MountingHole
Other:
- moved on the sheet: C1, C2, D1, D2, J1, J2, J3, R1, R2, R3, U1
